File: rc2014-ds1302-rtc.kicad_sch (KiCad schematic)
At the start: 15 parts, among them P1 RC2014 BUS, SW1 SW_DIP_x06, U1 74HCT688, U2 74HCT125, U3 74HCT174, U4 DS1302, U5 74HCT32, Y1 Crystal

Commit message: Complete kicad 6 migration
Parts:
- added unit 5 of U2
- added unit 5 of U5
- BT1: footprint Battery_Holders:Keystone_106_1x20mm-CoinCell -> Battery:BatteryHolder_Keystone_106_1x20mm; symbol rc2014-ds1302-rtc-rescue:Battery_Cell -> Device:Battery_Cell
- C1, C2, C3, C4, C5: symbol rc2014-ds1302-rtc-rescue:C -> Device:C
- P1: symbol rc2014-ds1302-rtc-rescue:Conn_01x39 -> Connector_Generic:Conn_01x39
- RN1: symbol rc2014-ds1302-rtc-rescue:R_Network07 -> Device:R_Network07
- SW1: symbol rc2014-ds1302-rtc-rescue:SW_DIP_x06 -> Switch:SW_DIP_x06
- U1: footprint Housings_DIP:DIP-20_W7.62mm_Socket_LongPads -> Package_DIP:DIP-20_W7.62mm_Socket_LongPads; symbol rc2014-ds1302-rtc-rescue:74LS688 -> 74xx:74LS688
- U2: footprint Housings_DIP:DIP-14_W7.62mm_Socket_LongPads -> Package_DIP:DIP-14_W7.62mm_Socket_LongPads; symbol rc2014-ds1302-rtc-rescue:74LS125 -> 74xx:74LS125
- U3: footprint Housings_DIP:DIP-16_W7.62mm_Socket_LongPads -> Package_DIP:DIP-16_W7.62mm_Socket_LongPads; symbol rc2014-ds1302-rtc:74LS174 -> 74xx:74LS174
- U4: value DS1302 -> DS1302+; footprint Housings_DIP:DIP-8_W7.62mm_Socket_LongPads -> Package_DIP:DIP-8_W7.62mm_Socket_LongPads; symbol rc2014-ds1302-rtc-rescue:DS1302 -> Timer_RTC:DS1302+
- U5: footprint Housings_DIP:DIP-14_W7.62mm_Socket_LongPads -> Package_DIP:DIP-14_W7.62mm_Socket_LongPads; symbol rc2014-ds1302-rtc-rescue:74LS32 -> 74xx:74LS32
- Y1: footprint Crystals:Crystal_Round_d2.0mm_Vertical -> Crystal:Crystal_Round_D2.0mm_Vertical; symbol rc2014-ds1302-rtc-rescue:Crystal -> Device:Crystal
Connections:
- net GND: now also U2.7 (GND), U5.7 (GND); no longer U2.7 (GND), U2.7 (GND), U2.7 (GND), U2.7 (GND), U5.7 (GND), U5.7 (GND), U5.7 (GND), U5.7 (GND)
- net VCC: now also U2.14 (VCC), U5.14 (VCC); no longer U2.14 (VCC), U2.14 (VCC), U2.14 (VCC), U2.14 (VCC), U5.14 (VCC), U5.14 (VCC), U5.14 (VCC), U5.14 (VCC)
- net A0: no longer names the net of P1.16 (Pin_16)
- net A1: no longer names the net of P1.15 (Pin_15)
- net A10: no longer names the net of P1.6 (Pin_6)
- net A11: no longer names the net of P1.5 (Pin_5)
- net A12: no longer names the net of P1.4 (Pin_4)
- net A13: no longer names the net of P1.3 (Pin_3)
- net A14: no longer names the net of P1.2 (Pin_2)
- net A15: no longer names the net of P1.1 (Pin_1)
- net A8: no longer names the net of P1.8 (Pin_8)
- net A9: no longer names the net of P1.7 (Pin_7)
- net CLK: no longer names the net of P1.21 (Pin_21)
- net D1: no longer names the net of P1.28 (Pin_28)
- net INT: no longer names the net of P1.22 (Pin_22)
- net MREQ: no longer names the net of P1.23 (Pin_23)
- net RX: no longer names the net of P1.36 (Pin_36)
- net TX: no longer names the net of P1.35 (Pin_35)
Other:
- moved on the sheet: BT1, SW1, Y1
