File: rc2014-ds1302-rtc.kicad_sch (KiCad schematic)
At the start: 15 parts, among them P1 RC2014 BUS, SW1 SW_DIP_x06, U1 74HCT688, U2 74HCT125, U3 74HCT174, U4 DS1302+, U5 74HCT32, Y1 Crystal

Commit message: some updates for kicad 9 - still quite a lot of DRC failures
Parts:
- C1, C2, C3, C4, C5: footprint Capacitors_THT:C_Disc_D3.0mm_W2.0mm_P2.50mm -> Capacitor_THT:C_Disc_D3.0mm_W2.0mm_P2.50mm
- RN1: footprint Resistors_THT:R_Array_SIP8 -> Resistor_THT:R_Array_SIP8
- SW1: footprint Buttons_Switches_THT:SW_DIP_x6_W7.62mm_Slide -> Button_Switch_THT:SW_DIP_SPSTx06_Slide_9.78x17.42mm_W7.62mm_P2.54mm
- U4: footprint Package_DIP:DIP-8_W7.62mm_Socket_LongPads -> Package_DIP:DIP-8_W7.62mm
Connections:
- net /IORQ: no longer P1.26 (Pin_26)
- net /M1: no longer P1.19 (Pin_19)
- net /RD: no longer P1.25 (Pin_25)
- net /RESET: no longer P1.20 (Pin_20)
- net /RTC_RD: no longer U5.6
- net /RTC_WR: no longer U5.3
- net /WR: no longer P1.24 (Pin_24)
- new net /IORQ: P1.26 (Pin_26)
- new net /M1: P1.19 (Pin_19)
- new net /RD: P1.25 (Pin_25)
- new net /RESET: P1.20 (Pin_20)
- new net /RTC_RD: U5.6
- new net /RTC_WR: U5.3
- new net /WR: P1.24 (Pin_24)
